File: lestoFly2.sch (KiCad schematic (older format))
At the start: 43 parts, among them J1 Conn_01x02_Male, J10 Conn_01x07_Male, J2 Conn_01x06_Male, J3 Conn_Coaxial, J4 Micro_SD_Card_Det, J5 Conn_01x07_Male, J6 Conn_01x02_Male, J7 Conn_01x02_Male, J8 Conn_01x02_Male, J9 Conn_01x02_Male, Q1 DMN6140L, U1 NCP1117-1.8_TO252, U2 STM32H743ZITx, U3 ICM-20948, U4 ICM-20948, U5 RFM95W-868S2, U6 BMP280, Y1 25MHz

Commit message: varius fixes
Parts:
- removed C16: 100nF, Capacitor_SMD:C_0603_1608Metric, symbol Device:C
- removed J2: Conn_01x06_Male, Connector_PinHeader_1.00mm:PinHeader_1x06_P1.00mm_Vertical, symbol Connector:Conn_01x06_Male
- removed Q1: DMN6140L, Package_TO_SOT_SMD:SOT-23, symbol Transistor_FET:DMN6140L
- removed U1: NCP1117-1.8_TO252, Package_TO_SOT_SMD:TO-252-2, symbol Regulator_Linear:NCP1117-1.8_TO252
- removed Y1: 25MHz, Crystal:Crystal_SMD_0603-4Pin_6.0x3.5mm_HandSoldering, symbol Device:Crystal_GND24
- added C1, C10, C11, C12, C13, C14, C19, C2, C26, C6, C7, C8, C9: 100nF, Capacitor_SMD:C_0603_1608Metric, symbol Device:C
- added C20: 1nF, Capacitor_SMD:C_0603_1608Metric, symbol Device:C
- added C27: 1uF, Capacitor_SMD:C_0603_1608Metric, symbol Device:C
- added D1: D, Diode_SMD:D_1210_3225Metric, symbol Device:D
- added F1: Polyfuse, Fuse:Fuse_1210_3225Metric, symbol Device:Polyfuse
- added J1: Conn_01x05_Male, Connector_PinHeader_1.00mm:PinHeader_1x05_P1.00mm_Vertical, symbol Connector:Conn_01x05_Male
- added R10, R11, R12, R3, R4, R7, R8, R9: 47ohm, Resistor_SMD:R_0603_1608Metric, symbol Device:R
- added R5, R6: 1.5k, Resistor_SMD:R_0603_1608Metric, symbol Device:R
- added U4: R-78C1.8-1.0, Converter_DCDC:Converter_DCDC_RECOM_R-78E-0.5_THT, symbol Regulator_Switching:R-78C1.8-1.0
- C21: renamed from C1; footprint Capacitor_SMD:C_0603_1608Metric -> Resistor_SMD:R_0805_2012Metric
- C3, C4: value 3.9pF -> 100nF
- R1: renamed from R3; footprint Resistor_SMD:R_0805_2012Metric_Pad1.15x1.40mm_HandSolder -> Resistor_SMD:R_0603_1608Metric
- R13: renamed from R5; footprint Resistor_SMD:R_0805_2012Metric_Pad1.15x1.40mm_HandSolder -> Resistor_SMD:R_0603_1608Metric
- R14: renamed from R1; footprint Resistor_SMD:R_0805_2012Metric -> Resistor_SMD:R_0603_1608Metric
- R15: renamed from R2; footprint Resistor_SMD:R_0805_2012Metric -> Resistor_SMD:R_0603_1608Metric
- R2: renamed from R4; footprint Resistor_SMD:R_0805_2012Metric_Pad1.15x1.40mm_HandSolder -> Resistor_SMD:R_0603_1608Metric
- renumbered C6 to C15, C7 to C16, C8 to C22, C9 to C23, C2 to C24, C10 to C25, C11 to C28, C12 to C29, C13 to C30, C14 to C31, C15 to C32, J4 to J10, J5 to J2, J10 to J3, J6 to J4, J7 to J5, J8 to J6, J9 to J7, J1 to J8, J3 to J9, U2 to U1, U5 to U2, U4 to U5
Connections:
- net +1V8: now also C3.2, C4.2, R2.1, U1.32 (VREF+), C1.2, C10.2, C11.2, C12.2, C13.2, C14.2, C2.2, C26.2, C27.2, C6.2, C7.2, C8.2, C9.2, J1.1 (Pin_1), R5.2, R6.2, U4.3 (OUT)
- net BAT_SCALED: now also C20.1
- net GND: now also C3.1, C4.1, J8.2 (Pin_2), C1.1, C10.1, C11.1, C12.1, C13.1, C14.1, C19.1, C2.1, C20.2, C26.1, C27.1, C6.1, C7.1, C8.1, C9.1, D1.2 (A), J1.2 (Pin_2), U4.2 (GND); no longer C3.2, C4.2, R2.1
- net I2C1_SCL: now also R5.1
- net I2C1_SDA: now also R6.1
- net SWCLK: now also J1.4 (Pin_4), R4.1; no longer U1.109 (PA14)
- net SWDIO: now also J1.3 (Pin_3), R3.1; no longer U1.105 (PA13)
- net USART1_RX: now also R7.2; no longer J4.2 (Pin_2)
- net USART1_TX: now also R8.2; no longer J4.1 (Pin_1)
- net USART2_RX: now also R9.2; no longer J5.2 (Pin_2)
- net USART2_TX: now also R10.2; no longer J5.1 (Pin_1)
- net USART3_RX: now also R11.2; no longer J6.2 (Pin_2)
- net USART3_TX: now also R12.2; no longer J6.1 (Pin_1)
- net VCC: now also D1.1 (K), F1.1, U4.1 (IN); no longer J8.1 (Pin_1)
- net at R2.2, U1.25 (NRST): now also C19.2
- net at R1.2: now also J1.5 (Pin_5)
- net at U1.23 (PH0): no longer C4.1
- net at U1.24 (PH1): no longer C3.1
- new net: R3.2, U1.105 (PA13)
- new net: R4.2, U1.109 (PA14)
- new net: F1.2, J8.1 (Pin_1)
- new net: J4.1 (Pin_1), R8.1
- new net: J4.2 (Pin_2), R7.1
- new net: J5.1 (Pin_1), R10.1
- new net: J5.2 (Pin_2), R9.1
- new net: J6.1 (Pin_1), R12.1
- new net: J6.2 (Pin_2), R11.1
- no-connect marks 81 -> 83
Other:
- moved on the sheet: C15, C16, R2
