File: lestoFly.kicad_pcb (KiCad board)
At the start: 2 copper layers, 36 x 36 mm, 25 parts, among them J1 Conn_01x02_Male, J2 Conn_01x04_Male, J3 Conn_01x05_Male, J4 Conn_01x03_Male, J5 Conn_Coaxial, U1 ESP32-WROOM-32D, U2 LMZM23601V3, U3 BMP280, U4 RFM95W-868S2, U5 BMX160

Commit message: board pcb redraw
Parts:
- C10, C6, C7, C8, C9, J5, U3, U4, U5: moved to B.Cu
- J2, J3, U1: moved to F.Cu
- moved C3 46.4 mm to (99.5, 61.0), turned to 90 degrees
- moved D2 46.0 mm to (114.0, 79.7), turned to 90 degrees
- moved C5 44.5 mm to (112.5, 79.7), turned to 90 degrees
- moved C8 43.6 mm to (118.0, 76.2)
- moved C1 42.7 mm to (99.5, 64.3)
- moved U2 41.6 mm to (109.5, 79.5), turned to 0 degrees
- moved R3 41.2 mm to (106.0, 79.6), turned to 270 degrees
- moved J2 39.7 mm to (122.0, 61.0)
- moved C2 39.3 mm to (99.5, 67.5), turned to 90 degrees
- moved J1 37.8 mm to (98.0, 75.5)
- moved D1 36.3 mm to (100.0, 76.0), turned to 270 degrees
- moved R2 35.4 mm to (104.0, 79.6), turned to 90 degrees
- moved U1 35.0 mm to (111.0, 67.0)
- moved C4 33.9 mm to (100.6, 79.5)
- moved J5 31.8 mm to (101.0, 79.0), turned to 0 degrees
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Connections:
- U1 pad 23: Net-(J3-Pad5) -> Net-(U1-Pad23)
Routing:
- net +3V3: track 81.9 -> 98.7 mm, vias 1 -> 2
- net CLK: track 34.4 -> 48.4 mm
- net Net-(J3-Pad5): track 12.7 -> 0.00 mm
- net MOSI: track 38.3 -> 50.3 mm
- net CS_IMU: track 14.1 -> 24.5 mm
- net MISO: track 35.7 -> 44.5 mm, vias 2 -> 1
- net INT_IMU: track 17.2 -> 24.4 mm
- net Net-(J3-Pad1): track 9.72 -> 2.57 mm
- net BAT_SCALED: track 9.35 -> 16.2 mm, vias 1 -> 0
- net Net-(J3-Pad2): track 9.45 -> 2.68 mm
- net Net-(J4-Pad1): track 9.80 -> 3.24 mm
- net Net-(J3-Pad3): track 9.18 -> 2.80 mm
- net CS_BARO: track 10.4 -> 16.8 mm
- net Net-(J3-Pad4): track 8.47 -> 2.91 mm
- net Net-(J4-Pad2): track 8.19 -> 2.76 mm
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Other:
- board size 36 x 36 mm -> 24 x 25 mm
- net class Default: clearance 0.15 -> 0.1
- rule trace_clearance: 0.15 -> 0.1

Commit message: new review finish
Parts:
- removed J3: Conn_01x05_Male, Connector_PinHeader_1.00mm:PinHeader_1x05_P1.00mm_Vertical
- removed J4: Conn_01x03_Male, Connector_PinHeader_1.00mm:PinHeader_1x03_P1.00mm_Vertical
- added R4: 10k, Resistor_SMD:R_0805_2012Metric, F.Cu at (88.0, 60.2)
- added REF**: OSHW-Logo2_7.3x6mm_Copper, Symbol:OSHW-Logo2_7.3x6mm_Copper, B.Cu at (97.5, 45.6)
- C10, C6, C7, C8, C9, J5, U3, U4, U5: moved to F.Cu
- J2: value Conn_01x04_Male -> Conn_01x15_Male; footprint Connector_PinHeader_1.00mm:PinHeader_1x04_P1.00mm_Vertical -> Connector_PinHeader_1.00mm:PinHeader_1x15_P1.00mm_Vertical
- U1: moved to B.Cu
- moved C8 35.5 mm to (107.8, 42.2), turned to 270 degrees
- moved C7 33.8 mm to (91.6, 59.3), turned to 90 degrees
- moved C10 33.8 mm to (93.1, 59.3), turned to 90 degrees
- moved U5 28.5 mm to (95.9, 59.3), turned to 180 degrees
- moved C5 24.7 mm to (91.5, 66.7), turned to 270 degrees
- moved D2 24.7 mm to (93.0, 66.7), turned to 270 degrees
- moved U3 23.3 mm to (99.8, 59.5), turned to 90 degrees
- moved U4 21.6 mm to (96.2, 48.9), turned to 0 degrees
- moved U2 19.4 mm to (95.6, 66.0), turned to 90 degrees
- moved J5 19.3 mm to (103.7, 59.8), turned to 180 degrees
- moved U1 16.4 mm to (96.6, 59.2)
- moved R3 15.9 mm to (99.3, 65.2), turned to 0 degrees
- moved J2 14.6 mm to (107.8, 64.0), turned to 180 degrees
- moved C4 13.8 mm to (102.8, 65.8), turned to 90 degrees
- moved R2 13.2 mm to (99.3, 67.2), turned to 180 degrees
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Connections:
- J2 pad 1: Net-(J2-Pad1) -> 1
- J2 pad 2: Net-(J2-Pad2) -> 2
- U1 pad 24: Net-(U1-Pad24) -> 15
- U1 pad 25: Net-(U1-Pad25) -> 14
- U1 pad 26: Net-(J3-Pad4) -> 13
- U1 pad 27: Net-(J3-Pad3) -> 12
- U1 pad 28: Net-(J3-Pad2) -> 11
- U1 pad 29: Net-(J3-Pad1) -> 10
- U1 pad 30: Net-(J4-Pad3) -> 9
- U1 pad 31: Net-(J4-Pad2) -> 8
- U1 pad 33: Net-(J4-Pad1) -> 7
- U1 pad 34: Net-(J2-Pad2) -> 6
- U1 pad 35: Net-(J2-Pad1) -> 5
- U1 pad 36: Net-(U1-Pad36) -> 2
- U1 pad 37: Net-(U1-Pad37) -> 1
- U5 pad 2: Net-(U5-Pad2) -> GND
- U5 pad 3: Net-(U5-Pad3) -> GND
Routing:
- net GND: track 39.7 -> 3.58 mm, vias 5 -> 1
- net +3V3: track 98.7 -> 76.4 mm, vias 2 -> 1
- net MOSI: track 50.3 -> 28.8 mm
- net CLK: track 48.4 -> 29.4 mm
- net CS_LORA: track 23.3 -> 6.23 mm
- net CS_IMU: track 24.5 -> 11.6 mm
- net MISO: track 44.5 -> 32.5 mm, vias 1 -> 3
- net Net-(R4-Pad1): track 0.00 -> 8.62 mm
- net Net-(C2-Pad1): track 10.4 -> 4.56 mm, vias 0 -> 1
- net 15: track 0.00 -> 5.45 mm
- net 5: track 0.00 -> 5.01 mm
- net 6: track 0.00 -> 4.74 mm
- net 7: track 0.00 -> 4.47 mm
- net 1: track 0.00 -> 3.84 mm
- net INT_IMU: track 24.4 -> 20.8 mm
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Other:
- board size 24 x 25 mm -> 23 x 29 mm
- net class Default: clearance 0.1 -> 0.15; trace_width 0.25 -> 0.15; via_dia 0.8 -> 0.6; via_drill 0.4 -> 0.35
- rule trace_clearance: 0.1 -> 0.15
- rule trace_min: 0.2 -> 0.15
- rule via_min_drill: 0.3 -> 0.35
- rule via_min_size: 0.4 -> 0.6
- board text added: "github.com/mauromombelli/lestoFly"

Commit message: completed lestoFly2
Parts:
- moved C8 4.82 mm to (106.8, 46.9), turned to 90 degrees
Routing:
- net +3V3: track 76.4 -> 70.8 mm
Changed lines of the file:
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@@
     (thickness 1.6)
     (drawings 2)
-    (tracks 272)
+    (tracks 270)
     (zones 0)
     (modules 25)
@@
   )
   (setup
-    (last_trace_width 0.15)
+    (last_trace_width 0.25)
+    (user_trace_width 0.15)
+    (user_trace_width 0.25)
     (trace_clearance 0.15)
     (zone_clearance 0.1)
@@
   )
   (module Capacitor_SMD:C_0603_1608Metric (layer F.Cu)
-    (at 107.75 42.2125 270)
+    (at 106.8 46.9375 90)
     (descr "Capacitor SMD 0603 (1608 Metric), square (rectangular) end terminal, IPC_7351 nominal, (Body size source: http://www.tortai-tech.com/upload/download/2011102023233369053.pdf), generated with kicad-footprint-generator")
     (tags capacitor)
@@
     (fp_line (start -0.8 -0.4) (end 0.8 -0.4) (layer F.Fab) (width 0.1))
     (fp_line (start -0.8 0.4) (end -0.8 -0.4) (layer F.Fab) (width 0.1))
-    (pad 2 smd roundrect (at 0.7875 0 270) (size 0.875 0.95) (layers F.Cu F.Paste F.Mask) (roundrect_rratio 0.25)
-      (net 1 GND))
-    (pad 1 smd roundrect (at -0.7875 0 270) (size 0.875 0.95) (layers F.Cu F.Paste F.Mask) (roundrect_rratio 0.25)
+    (pad 2 smd roundrect (at 0.7875 0 90) (size 0.875 0.95) (layers F.Cu F.Paste F.Mask) (roundrect_rratio 0.25)
+      (net 1 GND))
+    (pad 1 smd roundrect (at -0.7875 0 90) (size 0.875 0.95) (layers F.Cu F.Paste F.Mask) (roundrect_rratio 0.25)
       (net 2 +3V3))
     (model ${KISYS3DMOD}/Capacitor_SMD.3dshapes/C_0603_1608Metric.wrl
@@
   (segment (start 101.045001 59.119999) (end 101.045001 57.193721) (width 0.15) (layer F.Cu) (net 2))
   (segment (start 100.57 59.195) (end 100.97 59.195) (width 0.15) (layer F.Cu) (net 2) (status 10))
-  (segment (start 106.25 46.4) (end 104.75 47.9) (width 0.15) (layer F.Cu) (net 2) (status 20))
-  (segment (start 107.75 41.425) (end 106.25 42.925) (width 0.15) (layer F.Cu) (net 2) (status 10))
-  (segment (start 104.75 47.9) (end 104.25 47.9) (width 0.15) (layer F.Cu) (net 2) (status 30))
-  (segment (start 106.25 42.925) (end 106.25 46.4) (width 0.15) (layer F.Cu) (net 2))
+  (segment (start 106.625 47.9) (end 106.8 47.725) (width 0.15) (layer F.Cu) (net 2))
+  (segment (start 104.25 47.9) (end 106.625 47.9) (width 0.15) (layer F.Cu) (net 2))
   (segment (start 90.25773 64.1) (end 89.92442 64.43331) (width 0.15) (layer F.Cu) (net 3))
   (segment (start 89.48773 64.87) (end 89.92442 64.43331) (width 0.15) (layer B.Cu) (net 3))
@@
   (segment (start 103.685 56.465) (end 104.25 55.9) (width 0.15) (layer F.Cu) (net 6) (status 20))
   (segment (start 103.685 58.34) (end 103.685 56.465) (width 0.15) (layer F.Cu) (net 6) (status 10))
-  (segment (start 107.65 50.9) (end 107.75 51) (width 0.15) (layer B.Cu) (net 41) (status 30))
-  (segment (start 105.13 50.9) (end 107.65 50.9) (width 0.15) (layer B.Cu) (net 41) (status 30))
-  (segment (start 105.3 52) (end 105.13 52.17) (width 0.15) (layer B.Cu) (net 42) (status 30))
-  (segment (start 107.75 52) (end 105.3 52) (width 0.15) (layer B.Cu) (net 42) (status 30))
-  (segment (start 105.13 53.44) (end 106.49 53.44) (width 0.15) (layer B.Cu) (net 43) (status 10))
-  (segment (start 106.93 53) (end 107.75 53) (width 0.15) (layer B.Cu) (net 43) (status 20))
-  (segment (start 106.49 53.44) (end 106.93 53) (width 0.15) (layer B.Cu) (net 43))
-  (segment (start 106.43896 54.71) (end 105.13 54.71) (width 0.15) (layer B.Cu) (net 44) (status 20))
-  (segment (start 107.14896 54) (end 106.43896 54.71) (width 0.15) (layer B.Cu) (net 44))
-  (segment (start 107.75 54) (end 107.14896 54) (width 0.15) (layer B.Cu) (net 44) (status 10))
   (segment (start 98.35 67.2) (end 98.35 65.2) (width 0.15) (layer F.Cu) (net 7) (status 30))
   (segment (start 89.66 61.31) (end 90.34 61.99) (width 0.15) (layer F.Cu) (net 7))
@@
   (segment (start 107.65 49.9) (end 107.75 50) (width 0.15) (layer B.Cu) (net 40) (status 30))
   (segment (start 102.345 49.9) (end 107.65 49.9) (width 0.15) (layer B.Cu) (net 40) (status 30))
+  (segment (start 107.65 50.9) (end 107.75 51) (width 0.15) (layer B.Cu) (net 41) (status 30))
+  (segment (start 105.13 50.9) (end 107.65 50.9) (width 0.15) (layer B.Cu) (net 41) (status 30))
+  (segment (start 105.3 52) (end 105.13 52.17) (width 0.15) (layer B.Cu) (net 42) (status 30))
+  (segment (start 107.75 52) (end 105.3 52) (width 0.15) (layer B.Cu) (net 42) (status 30))
+  (segment (start 105.13 53.44) (end 106.49 53.44) (width 0.15) (layer B.Cu) (net 43) (status 10))
+  (segment (start 106.93 53) (end 107.75 53) (width 0.15) (layer B.Cu) (net 43) (status 20))
+  (segment (start 106.49 53.44) (end 106.93 53) (width 0.15) (layer B.Cu) (net 43))
+  (segment (start 106.43896 54.71) (end 105.13 54.71) (width 0.15) (layer B.Cu) (net 44) (status 20))
+  (segment (start 107.14896 54) (end 106.43896 54.71) (width 0.15) (layer B.Cu) (net 44))
+  (segment (start 107.75 54) (end 107.14896 54) (width 0.15) (layer B.Cu) (net 44) (status 10))
   (segment (start 106.77 55.98) (end 107.75 55) (width 0.15) (layer B.Cu) (net 45))
   (segment (start 105.13 55.98) (end 106.77 55.98) (width 0.15) (layer B.Cu) (net 45))

Commit message: revived esp32
Parts:
- removed REF**: OSHW-Logo2_7.3x6mm_Copper, Symbol:OSHW-Logo2_7.3x6mm_Copper

Commit message: completed the esp32 version
Parts:
- removed the C8 at (106.8, 46.9)
- removed D1: DIODE, Diode_SMD:D_0603_1608Metric
- removed D2: D_Zener, Diode_SMD:D_0603_1608Metric
- removed J2: Conn_01x15_Male, Connector_PinHeader_1.00mm:PinHeader_1x15_P1.00mm_Vertical
- removed R4: 10k, Resistor_SMD:R_0805_2012Metric
- removed U4: RFM95W-868S2, RF_Module:HOPERF_RFM9XW_SMD
- added C10: 100nF, Capacitor_SMD:C_0603_1608Metric, F.Cu at (93.0, 68.0)
- added C5: 100nF, Capacitor_SMD:C_0603_1608Metric, F.Cu at (104.2, 51.9)
- added C6: 10uF, Capacitor_SMD:C_0603_1608Metric, F.Cu at (102.7, 51.9)
- added C9: 100nF, Capacitor_SMD:C_0603_1608Metric, F.Cu at (90.0, 64.4)
- added G***: LOGO, lestoFly:oshw_2.0x1, F.Cu at (108.1, 59.5)
- added J3: Conn_01x04_Male, Connector_PinHeader_1.00mm:PinHeader_1x04_P1.00mm_Vertical, F.Cu at (108.3, 64.6)
- added J4: Conn_01x04_Male, lestoFly:PinHeader_1x04_P1.00mm_Vertical_small, F.Cu at (108.4, 57.0)
- added Q1: ZXMP6A13F, Package_TO_SOT_SMD:SOT-23, F.Cu at (105.4, 64.9)
- added R5: 12K, Capacitor_SMD:C_0603_1608Metric, F.Cu at (105.6, 67.4)
- added U6: BMX160, Package_LGA:LGA-14_3x2.5mm_P0.5mm_LayoutBorder3x4y, F.Cu at (90.0, 67.0)
- C13: renamed from C2; value 0.1uF -> 100nF
- C3: renamed from C4; value 10uF -> 0.1uF
- C4: renamed from C5; value 33uF -> 0.1uF
- J5: value Conn_Coaxial -> Micro_SD_Card_Det; footprint Connector_Coaxial:U.FL_Molex_MCRF_73412-0110_Vertical -> Connector_Card:microSD_HC_Hirose_DM3D-SF
- U2: value LMZM23601V3 -> LM3480-3.3; footprint Package_LGA:Texas_SIL0010A_MicroSiP-10-1EP_3.8x3mm_P0.6mm_EP0.7x2.9mm_ThermalVias -> Package_TO_SOT_SMD:SOT-23
- moved C11 15.5 mm to (103.7, 49.7), turned to 0 degrees
- moved C12 14.9 mm to (106.9, 53.6), turned to 270 degrees
- moved U5 14.3 mm to (107.0, 50.4), turned to 90 degrees
- moved J5 9.89 mm to (95.0, 55.0)
- moved C2 9.68 mm to (97.6, 63.4), turned to 0 degrees
- moved C8 8.28 mm to (105.4, 56.1)
- moved R2 8.08 mm to (104.9, 61.4), turned to 90 degrees
- moved C7 6.36 mm to (103.5, 58.4), turned to 180 degrees
- moved R3 5.28 mm to (103.0, 61.4), turned to 270 degrees
- moved C13 5.18 mm to (93.3, 64.6), turned to 0 degrees
- moved U3 4.97 mm to (103.3, 56.1)
- moved C1 4.68 mm to (90.0, 62.5)
- moved C4 3.89 mm to (95.3, 66.9)
- moved U2 2.83 mm to (98.4, 66.4)
- moved R1 1.89 mm to (93.5, 62.8)
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- renumbered C7 to C11, C10 to C12, C3 to C2, C6 to C7, C9 to C8
Connections:
- J5 pad 1: Net-(J5-Pad1) -> SD_DAT2
- J5 pad 2: GND -> SD_DAT3
- U1 pad 10: CS_IMU -> CS_IMU_1
- U1 pad 12: CS_LORA -> Net-(U1-Pad12)
- U1 pad 13: CLK -> SD_CLK
- U1 pad 14: MISO -> SD_DAT2
- U1 pad 16: MOSI -> SD_DAT3
- U1 pad 23: Net-(U1-Pad23) -> SD_CMD
- U1 pad 24: 15 -> SD_DAT0
- U1 pad 25: 14 -> 7
- U1 pad 26: 13 -> SD_DAT1
- U1 pad 27: 12 -> INT_IMU_2
- U1 pad 28: 11 -> 6
- U1 pad 29: 10 -> 5
- U1 pad 30: 9 -> CLK
- U1 pad 31: 8 -> MISO
- U1 pad 33: 7 -> 4
- U1 pad 34: 6 -> 3
- U1 pad 35: 5 -> 2
- U1 pad 36: 2 -> 1
- U1 pad 37: 1 -> MOSI
- U1 pad 6: INT_IMU -> INT_IMU_1
- U1 pad 8: Net-(U1-Pad8) -> CS_IMU_2
- U2 pad 1: GND -> +3V3
- U2 pad 3: VCC -> GND
- U5 pad 12: CS_IMU -> CS_IMU_2
- U5 pad 4: INT_IMU -> INT_IMU_2
Routing:
- net CS_IMU_2: track 0.00 -> 22.2 mm, vias 0 -> 1
- net INT_IMU: track 20.8 -> 0.00 mm, vias 1 -> 0
- net CS_IMU_1: track 0.00 -> 17.4 mm, vias 0 -> 1
- net +3V3: track 70.8 -> 87.9 mm, vias 1 -> 7
- net SD_CMD: track 0.00 -> 12.6 mm, vias 0 -> 1
- net CS_IMU: track 11.6 -> 0.00 mm, vias 1 -> 0
- net MOSI: track 28.8 -> 39.0 mm
- net SD_DAT1: track 0.00 -> 10.0 mm, vias 0 -> 1
- net SD_CLK: track 0.00 -> 9.08 mm, vias 0 -> 1
- net Net-(R4-Pad1): track 8.62 -> 0.00 mm
- net SD_DAT0: track 0.00 -> 7.96 mm, vias 0 -> 1
- net INT_IMU_1: track 0.00 -> 7.58 mm, vias 0 -> 1
- net GND: track 3.58 -> 10.8 mm, vias 1 -> 29
- net CS_LORA: track 6.23 -> 0.00 mm, vias 1 -> 0
- net 15: track 5.45 -> 0.00 mm
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Other:
- board size 23 x 29 mm -> 21 x 21 mm
- board text added: "lestoFly"
- board text removed: "github.com/mauromombelli/lestoFly"
