File: lestoFly.sch (KiCad schematic (older format))
At the start: 25 parts, among them J1 Conn_01x02_Male, J2 Conn_01x04_Male, J3 Conn_01x05_Male, J4 Conn_01x03_Male, J5 Conn_Coaxial, U1 ESP32-WROOM-32D, U2 LMZM23601V3, U3 BMP280, U4 RFM95W-868S2, U5 BMX160

Commit message: board pcb redraw
Connections:
- wire segments 91 -> 88
Changed lines of the file:
@@
-	1    0    0    -1
-$EndComp
-$Comp
-L Device:C C4
-U 1 1 5CFBA42A
-P 2000 1850
-F 0 "C4" H 2115 1896 50  0000 L CNN
-F 1 "10uF" H 2115 1805 50  0000 L CNN
-F 2 "Capacitor_SMD:C_1210_3225Metric" H 2038 1700 50  0001 C CNN
-F 3 "~" H 2000 1850 50  0001 C CNN
-	1    2000 1850
 	1    0    0    -1
 $EndComp
@@
 Text GLabel 3300 4900 2    50   Input ~ 0
 MISO
-Text GLabel 3300 5000 2    50   Input ~ 0
-MOSI
 Text GLabel 3300 5100 2    50   Input ~ 0
 CLK
@@
 	1300 2300 2000 2300
 Wire Wire Line
-	3000 5200 3600 5200
-Wire Wire Line
-	3600 5200 3600 5000
-Wire Wire Line
-	3600 5000 4100 5000
-Wire Wire Line
 	3000 4700 3850 4700
 Wire Wire Line
@@
 Text GLabel 3300 6000 2    50   Output ~ 0
 CS_IMU
+$Comp
+L Device:C C4
+U 1 1 5CFBA42A
+P 2000 1850
+F 0 "C4" H 2115 1896 50  0000 L CNN
+F 1 "10uF" H 2115 1805 50  0000 L CNN
+F 2 "Capacitor_SMD:C_1210_3225Metric" H 2038 1700 50  0001 C CNN
+F 3 "~" H 2000 1850 50  0001 C CNN
+	1    2000 1850
+	1    0    0    -1
+$EndComp
+Text GLabel 3300 5000 2    50   Input ~ 0
+MOSI
 $EndSCHEMATC

Commit message: new review finish
Parts:
- removed J2: Conn_01x04_Male, Connector_PinHeader_1.00mm:PinHeader_1x04_P1.00mm_Vertical, symbol Connector:Conn_01x04_Male
- removed J3: Conn_01x05_Male, Connector_PinHeader_1.00mm:PinHeader_1x05_P1.00mm_Vertical, symbol Connector:Conn_01x05_Male
- removed J4: Conn_01x03_Male, Connector_PinHeader_1.00mm:PinHeader_1x03_P1.00mm_Vertical, symbol Connector:Conn_01x03_Male
- added J2: Conn_01x15_Male, Connector_PinHeader_1.00mm:PinHeader_1x15_P1.00mm_Vertical, symbol Connector:Conn_01x15_Male
- added R4: 10k, Resistor_SMD:R_0805_2012Metric, symbol Device:R
Connections:
- net labels added: 1, 10, 11, 12, 13, 14, 15, 2, 5, 6, 7, 8, 9
- wire segments 88 -> 75
- no-connect marks 0 -> 19

Commit message: completed lestoFly2
Parts:
- C2: value 0.1uF -> 100nF
Changed lines of the file:
@@
 P 1350 4550
 F 0 "C2" H 1465 4596 50  0000 L CNN
-F 1 "0.1uF" H 1465 4505 50  0000 L CNN
+F 1 "100nF" H 1465 4505 50  0000 L CNN
 F 2 "Capacitor_SMD:C_0603_1608Metric" H 1388 4400 50  0001 C CNN
 F 3 "~" H 1350 4550 50  0001 C CNN

Commit message: revived esp32
Parts:
- removed C8: 100nF, Capacitor_SMD:C_0603_1608Metric, symbol Device:C
- removed D1: DIODE, Diode_SMD:D_0603_1608Metric, symbol pspice:DIODE
- removed D2: D_Zener, Diode_SMD:D_0603_1608Metric, symbol Device:D_Zener
- removed J5: Conn_Coaxial, Connector_Coaxial:U.FL_Molex_MCRF_73412-0110_Vertical, symbol Connector:Conn_Coaxial
- removed R4: 10k, Resistor_SMD:R_0805_2012Metric, symbol Device:R
- removed U4: RFM95W-868S2, RF_Module:HOPERF_RFM9XW_SMD, symbol RF_Module:RFM95W-868S2
- added C11, C12: 100nF, Capacitor_SMD:C_0603_1608Metric, symbol Device:C
- added J3: Micro_SD_Card_Det, Connector_Card:microSD_HC_Hirose_DM3D-SF, symbol Connector:Micro_SD_Card_Det
- added Q1: ZXMP6A13F, Package_TO_SOT_SMD:SOT-23, symbol Device:Q_PMOS_SGD
- added R5: 12K, Capacitor_SMD:C_0603_1608Metric, symbol Device:R
- added U6: BMX160, Package_LGA:LGA-14_3x2.5mm_P0.5mm_LayoutBorder3x4y, symbol lesto:BMX160
Connections:
- net labels added: 3, 4, CS_IMU_1, CS_IMU_2, SD_CLK, SD_CMD, SD_DAT0, SD_DAT1, SD_DAT2, SD_DAT3
- net labels removed: CS_IMU, CS_LORA
- wire segments 75 -> 100
- no-connect marks 19 -> 13
Other:
- note removed: "LORA"
- moved on the sheet: C6, C9, R2, R3, U3

Commit message: completed the esp32 version
Parts:
- removed J2: Conn_01x15_Male, Connector_PinHeader_1.00mm:PinHeader_1x15_P1.00mm_Vertical, symbol Connector:Conn_01x15_Male
- removed U2: LMZM23601V3, Package_LGA:Texas_SIL0010A_MicroSiP-10-1EP_3.8x3mm_P0.6mm_EP0.7x2.9mm_ThermalVias, symbol Regulator_Switching:LMZM23601V3
- added C5: 100nF, Capacitor_SMD:C_0603_1608Metric, symbol Device:C
- added C6: 10uF, Capacitor_SMD:C_0603_1608Metric, symbol Device:C
- added J3: Conn_01x04_Male, Connector_PinHeader_1.00mm:PinHeader_1x04_P1.00mm_Vertical, symbol Connector:Conn_01x04_Male
- added J4: Conn_01x04_Male, lestoFly:PinHeader_1x04_P1.00mm_Vertical_small, symbol Connector:Conn_01x04_Male
- added U2: LM3480-3.3, Package_TO_SOT_SMD:SOT-23, symbol Regulator_Linear:LM3480-3.3
- C3: renamed from C4; value 10uF -> 0.1uF
- C4: renamed from C5; value 33uF -> 0.1uF
- renumbered C12 to C10, C7 to C11, C10 to C12, C2 to C13, C3 to C2, C6 to C7, C9 to C8, C11 to C9, J3 to J5
Connections:
- net labels added: INT_IMU_1, INT_IMU_2
- net labels removed: 10, 11, 12, 13, 14, 15, 8, 9, INT_IMU
- wire segments 100 -> 105
- no-connect marks 13 -> 15
